File: xiaomao.kicad_sch (KiCad schematic)
At the start: 52 parts, among them J1 USB, J2 SWD, J4 USB_C_Receptacle_USB2.0, J5 JTAG, J6 UART, SW2 USB_BOOT, SW3 RESET, U1 HE6206-33NR, U2 W25Q128JVP, U3 RP2040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

Commit message: updating part numbers and lcsc numbers to those used in prototype
Parts:
- C1, C2: LCSC C106203 -> C1555; P/N CC0402JRNPO9BN220 -> 0402CG220J500NT; mfg YAGEO -> (none)
- C11, C12, C13, C14, C15, C19, C4, C6, C7, C9: LCSC C100072 -> C1525; P/N CL05A104KA5NNNC -> CL05B104KO5NNNC
- FB1: LCSC C76886 -> C1002; P/N BLM15AX601SN1D -> GZ1608D601TF; mfg Murata -> (none)
- J1: now not fitted
- J4: P/N USB-TYPE-C-018 -> USB-TYPE-C-018
- J5: LCSC C225494 -> C706871; P/N (none) -> X6511WR-08H-C60D30R2
- J6: LCSC C225495 -> C706872; P/N (none) -> X6511WR-09H-C60D30R2
- R10, R11, R13, R14, R15, R16, R17, R18, R19, R2, R20, R6, R9: P/N (none) -> 0603WAF2000T5E
- R7, R8: LCSC C25941 -> C25905; P/N 0402WGJ0512TCE -> 0402WGF5101TCE
- U1: LCSC C5199441 -> C5446; P/N HE6206-33NR -> XC6206P332MR-G; mfg HEERMICR -> (none)
Changed lines of the file:
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@@
 		(in_bom yes)
 		(on_board yes)
-		(dnp no)
+		(dnp yes)
 		(property "Reference" "J1"
 			(at 127 63.5 0)
@@
 			)
 		)
-		(property "LCSC" "C100072"
+		(property "LCSC" "C1525"
 			(at 262.89 25.4 0)
 			(effects
@@
 			)
 		)
-		(property "P/N" "CL05A104KA5NNNC"
+		(property "P/N" "CL05B104KO5NNNC"
 			(at 262.89 25.4 0)
 			(effects
@@
 			)
 		)
+		(property "P/N" "0603WAF2000T5E"
+			(at 107.95 170.18 0)
+			(effects
+				(font
+					(size 1.27 1.27)
+				)
+				(hide yes)
+			)
+		)
 		(pin "2"
 		)
@@
 			)
 		)
-		(property "P/N" "0402WGJ0512TCE"
+		(property "P/N" "0402WGF5101TCE"
 			(at 50.8 39.37 90)
 			(effects
@@
 			)
 		)
-		(property "LCSC" "C25941"
+		(property "LCSC" "C25905"
 			(at 50.8 39.37 90)
 			(effects
@@
 			)
 		)
+		(property "P/N" "0603WAF2000T5E"
+			(at 71.12 177.8 0)
+			(effects
+				(font
+					(size 1.27 1.27)
+				)
+				(hide yes)
+			)
+		)
 		(pin "1"
 		)
@@
 			)
 		)
+		(property "P/N" "0603WAF2000T5E"
+			(at 107.95 177.8 0)
+			(effects
+				(font
+					(size 1.27 1.27)
+				)
+				(hide yes)
+			)
+		)
 		(pin "2"
 		)
@@
 			)
 		)
-		(property "P/N" " USB-TYPE-C-018"
+		(property "P/N" "USB-TYPE-C-018"
 			(at 31.75 46.99 0)
 			(effects
@@
 			)
 		)
-		(property "LCSC" "C100072"
+		(property "LCSC" "C1525"
 			(at 179.07 25.4 0)
 			(effects
@@
 			)
 		)
-		(property "P/N" "CL05A104KA5NNNC"
+		(property "P/N" "CL05B104KO5NNNC"
 			(at 179.07 25.4 0)
 			(effects
@@
 			)
 		)
+		(property "P/N" "0603WAF2000T5E"
+			(at 107.95 175.26 0)
+			(effects
+				(font
+					(size 1.27 1.27)
+				)
+				(hide yes)
+			)
+		)
 		(pin "2"
 		)
@@
 			)
 		)
-		(property "LCSC" "C100072"
+		(property "LCSC" "C1525"
 			(at 222.25 25.4 0)
 			(effects
@@
 			)
 		)
-		(property "P/N" "CL05A104KA5NNNC"
+		(property "P/N" "CL05B104KO5NNNC"
 			(at 222.25 25.4 0)
 			(effects
@@
 			)
 		)
+		(property "P/N" "0603WAF2000T5E"
+			(at 71.12 172.72 0)
+			(effects
+				(font
+					(size 1.27 1.27)
+				)
+				(hide yes)
+			)
+		)
 		(pin "2"
 		)
@@
 			)
 		)
-		(property "LCSC" "C100072"
+		(property "LCSC" "C1525"
 			(at 242.57 25.4 0)
 			(effects
@@
 			)
 		)
-		(property "P/N" "CL05A104KA5NNNC"
+		(property "P/N" "CL05B104KO5NNNC"
 			(at 242.57 25.4 0)
 			(effects
@@
 			)
 		)
-		(property "LCSC" "C100072"
+		(property "LCSC" "C1525"
 			(at 120.65 102.87 0)
 			(effects
@@
 			)
 		)
-		(property "P/N" "CL05A104KA5NNNC"
+		(property "P/N" "CL05B104KO5NNNC"
 			(at 120.65 102.87 0)
 			(effects
@@
 			)
 		)
-		(property "P/N" "BLM15AX601SN1D"
+		(property "P/N" "GZ1608D601TF"
 			(at 55.88 29.21 90)
 			(effects
@@
 			)
 		)
-		(property "LCSC" "C76886"
+		(property "LCSC" "C1002"
 			(at 55.88 29.21 90)
 			(effects
@@
 			)
 		)
-		(property "mfg" "Murata"
+		(property "mfg" ""
 			(at 55.88 29.21 0)
 			(effects
@@
 			)
 		)
+		(property "P/N" "0603WAF2000T5E"
+			(at 71.12 165.1 0)
+			(effects
+				(font
+					(size 1.27 1.27)
+				)
+				(hide yes)
+			)
+		)
 		(pin "1"
 		)
@@
 			)
 		)
-		(property "LCSC" "C100072"
+		(property "LCSC" "C1525"
 			(at 273.05 25.4 0)
 			(effects
@@
 			)
 		)
-		(property "P/N" "CL05A104KA5NNNC"
+		(property "P/N" "CL05B104KO5NNNC"
 			(at 273.05 25.4 0)
 			(effects
@@
 			)
 		)
-		(property "P/N" "CL05A104KA5NNNC"
+		(property "P/N" "CL05B104KO5NNNC"
 			(at 63.5 34.29 0)
 			(effects
@@
 			)
 		)
-		(property "LCSC" "C100072"
+		(property "LCSC" "C1525"
 			(at 63.5 34.29 0)
 			(effects
@@
 			)
 		)
-		(property "P/N" "0402WGJ0512TCE"
+		(property "P/N" "0402WGF5101TCE"
 			(at 50.8 36.83 90)
 			(effects
@@
 			)
 		)
-		(property "LCSC" "C25941"
+		(property "LCSC" "C25905"
 			(at 50.8 36.83 90)
 			(effects
@@
 			)
 		)
+		(property "P/N" "0603WAF2000T5E"
+			(at 107.95 180.34 0)
+			(effects
+				(font
+					(size 1.27 1.27)
+				)
+				(hide yes)
+			)
+		)
 		(pin "2"
 		)
@@
 			)
 		)
+		(property "P/N" "0603WAF2000T5E"
+			(at 71.12 175.26 0)
+			(effects
+				(font
+					(size 1.27 1.27)
+				)
+				(hide yes)
+			)
+		)
 		(pin "1"
 		)
@@
 			)
 		)
+		(property "P/N" "0603WAF2000T5E"
+			(at 107.95 172.72 0)
+			(effects
+				(font
+					(size 1.27 1.27)
+				)
+				(hide yes)
+			)
+		)
 		(pin "1"
 		)
@@
 			)
 		)
-		(property "LCSC" "C100072"
+		(property "LCSC" "C1525"
 			(at 190.5 25.4 0)
 			(effects
@@
 			)
 		)
-		(property "P/N" "CL05A104KA5NNNC"
+		(property "P/N" "CL05B104KO5NNNC"
 			(at 190.5 25.4 0)
 			(effects
@@
 			)
 		)
-		(property "LCSC" "C100072"
+		(property "LCSC" "C1525"
 			(at 252.73 25.4 0)
 			(effects
@@
 			)
 		)
-		(property "P/N" "CL05A104KA5NNNC"
+		(property "P/N" "CL05B104KO5NNNC"
 			(at 252.73 25.4 0)
 			(effects
@@
 			)
 		)
-		(property "LCSC" "C100072"
+		(property "LCSC" "C1525"
 			(at 232.41 25.4 0)
 			(effects
@@
 			)
 		)
-		(property "P/N" "CL05A104KA5NNNC"
+		(property "P/N" "CL05B104KO5NNNC"
 			(at 232.41 25.4 0)
 			(effects
@@
 			)
 		)
-		(property "LCSC" "C5199441"
+		(property "LCSC" "C5446"
 			(at 102.87 29.21 0)
 			(effects
@@
 			)
 		)
-		(property "P/N" "HE6206-33NR"
+		(property "P/N" "XC6206P332MR-G "
 			(at 102.87 29.21 0)
 			(effects
@@
 			)
 		)
-		(property "mfg" "HEERMICR"
+		(property "mfg" ""
 			(at 102.87 29.21 0)
 			(effects
@@
 			)
 		)
+		(property "P/N" "0603WAF2000T5E"
+			(at 107.95 185.42 0)
+			(effects
+				(font
+					(size 1.27 1.27)
+				)
+				(hide yes)
+			)
+		)
 		(pin "2"
 		)
@@
 			)
 		)
+		(property "P/N" "0603WAF2000T5E"
+			(at 71.12 167.64 0)
+			(effects
+				(font
+					(size 1.27 1.27)
+				)
+				(hide yes)
+			)
+		)
 		(pin "1"
 		)
@@
 			)
 		)
-		(property "LCSC" "C225495"
+		(property "LCSC" "C706872"
+			(at 129.54 175.26 0)
+			(effects
+				(font
+					(size 1.27 1.27)
+				)
+				(hide yes)
+			)
+		)
+		(property "P/N" "X6511WR-09H-C60D30R2 "
 			(at 129.54 175.26 0)
 			(effects
@@
 			)
 		)
-		(property "LCSC" "C225494"
+		(property "LCSC" "C706871"
+			(at 53.34 172.72 0)
+			(effects
+				(font
+					(size 1.27 1.27)
+				)
+				(hide yes)
+			)
+		)
+		(property "P/N" "X6511WR-08H-C60D30R2 "
 			(at 53.34 172.72 0)
 			(effects
@@
 			)
 		)
+		(property "P/N" "0603WAF2000T5E"
+			(at 71.12 170.18 0)
+			(effects
+				(font
+					(size 1.27 1.27)
+				)
+				(hide yes)
+			)
+		)
 		(pin "1"
 		)
@@
 			)
 		)
-		(property "LCSC" "C106203"
+		(property "LCSC" "C1555"
 			(at 31.75 120.65 0)
 			(effects
@@
 			)
 		)
-		(property "P/N" "CC0402JRNPO9BN220"
+		(property "P/N" "0402CG220J500NT"
 			(at 31.75 120.65 0)
 			(effects
@@
 			)
 		)
-		(property "mfg" "YAGEO"
+		(property "mfg" ""
 			(at 31.75 120.65 0)
 			(effects
@@
 			)
 		)
+		(property "P/N" "0603WAF2000T5E"
+			(at 107.95 182.88 0)
+			(effects
+				(font
+					(size 1.27 1.27)
+				)
+				(hide yes)
+			)
+		)
 		(pin "2"
 		)
@@
 			)
 		)
-		(property "LCSC" "C106203"
+		(property "LCSC" "C1555"
 			(at 39.37 120.65 0)
 			(effects
@@
 			)
 		)
-		(property "P/N" "CC0402JRNPO9BN220"
+		(property "P/N" "0402CG220J500NT"
 			(at 39.37 120.65 0)
 			(effects
@@
 			)
 		)
-		(property "mfg" "YAGEO"
+		(property "mfg" ""
 			(at 39.37 120.65 0)
 			(effects
